File: kicad/winch_mainboard/winch_mainboard.kicad_pcb (KiCad board)
At the start: 2 copper layers, 180.5 x 114 mm, 38 parts, among them J1 PWR_IN_24V (from Victron 96V-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, J10 Heltec WiFi LoRa 32 V4 - Head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, J11 Heltec WiFi LoRa 32 V4 - Head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, J12 Hall sensors (drum direction), J2 CAN_BUS (to Fardriver), J3 To GIGA UART (TXD,RXD,GND), J4 HX711 module (3V3,GND,DT,SCK), J6 Spare I/O, J7 Line cut switch (winch), J8 Winchman remote switches, J9 Cut motor out (24V) - A/B = K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, K1 Relay 24V coil (Songle SRD-24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, Q1 BC337-40, U1 ESP32-S3 N16R8 DevKitC-1, U3 SN65HVD230

Commit message: update
Parts:
- added R31: 10k, Resistor_THT:R_Axial_DIN0207_L6.3mm_D2.5mm_P10.16mm_Horizontal, F.Cu at (32.5, 73.0)
- DCDC1: value DCDC 24V->5V module (MP1584) -> DCDC 24V->5V MP1584
- DCDC2: value DCDC 24V->3V3 module (MP1584) -> DCDC 24V->3V3 MP1584
- J1: value PWR_IN_24V (from Victron 96V->24V) -> PWR_IN_24V
- J10: value Heltec WiFi LoRa 32 V4 - Header J2 -> Heltec
- J11: value Heltec WiFi LoRa 32 V4 - Header J3 (reserved) -> Heltec
- J12: value Hall sensors (drum direction) -> Hall sensors drum
- J2: value CAN_BUS (to Fardriver) -> CAN_BUS Fardriver
- J3: value To GIGA UART (TXD,RXD,GND) -> GIGA UART (TXD,RXD,GND)
- J4: value HX711 module (3V3,GND,DT,SCK) -> HX711 module; footprint Connector_JST:JST_XH_B4B-XH-A_1x04_P2.50mm_Vertical -> Connector_PinSocket_2.54mm:PinSocket_1x04_P2.54mm_Vertical
- J7: value Line cut switch (winch) -> Line cut switch
- J9: value Cut motor out (24V) - A/B = K1 contacts, verify NO before wiring -> Cut motor out (24V)
- K1: value Relay 24V coil (Songle SRD-24VDC-SL-C) -> Songle SRD-24VDC-SL-C
- moved J4 1.12 mm to (99.0, 18.5), turned to 90 degrees
Connections:
- J4 pad 1: +3V3 -> GND
- J4 pad 2: GND -> HX711_DT
- J4 pad 3: HX711_DT -> HX711_SCK
- J4 pad 4: HX711_SCK -> +3V3
Routing:
- net ESTOP_SENSE: track 78.7 -> 143.5 mm, vias 0 -> 2
- net +3V3: track 395.2 -> 406.9 mm
- net +5V: track 379.0 -> 370.1 mm
- net HX711_DT: track 25.6 -> 27.6 mm
- net HX711_SCK: track 23.2 -> 25.2 mm
Other:
- board text added: "Paraglider-tow-winch 1.0"

Commit message: kicad: widen winchman remote (J8) to 7 pins for a proper release-switch pull-up, replacing the planned hand-wired bodge
J8 was full at 6/6 pins, so the release switch (added last session as a
firmware-only GPIO2 target) had no clean way to get a real pull-up like
the other four winchman-remote switches. Instead of the planned hand-wired
jumper off J6's spare pin, widened J8 to a 7-pin JST-XH connector and
added R35 (10k, +3V3 to SPARE_GPIO2/GPIO2) - same convention as R31-R34.

New Conn_01x07 schematic symbol (extended from the stock Conn_01x06
pattern, same pin pitch). PCB footprint swapped to the stock
JST_XH_B7B-XH-A_1x07; pins 1-6 keep identical physical positions so
existing routed copper is untouched. R35 placed at a location verified
clear of existing traces/footprints (an earlier attempt at a more
"obvious" spot turned out to short against an existing TENSION_RESET_SENSE
trace - moved after DRC caught it). back_gnd zone refilled to account for
the 3 new pads. ERC/DRC clean except pre-existing warnings and the 3 new
unrouted connections, left for manual routing as usual.

Also: .gitignore now excludes *.lck (KiCad's own transient lock files,
were being churned in/out of git status on every open/close).
Parts:
- added R35: 10k, Resistor_THT:R_Axial_DIN0207_L6.3mm_D2.5mm_P10.16mm_Horizontal, F.Cu at (100.0, 83.0)
- J8: footprint Connector_JST:JST_XH_B6B-XH-A_1x06_P2.50mm_Vertical -> Connector_JST:JST_XH_B7B-XH-A_1x07_P2.50mm_Vertical
Changed lines of the file:
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@@
+		)
+	)
+	(footprint "Resistor_THT:R_Axial_DIN0207_L6.3mm_D2.5mm_P10.16mm_Horizontal"
+		(layer "F.Cu")
+		(at 100 83)
+		(descr "Resistor, Axial_DIN0207 series, Axial, Horizontal, pin pitch=10.16mm, 0.25W = 1/4W, length*diameter=6.3*2.5mm^2, http://cdn-reichelt.de/documents/datenblatt/B400/1_4W%23YAG.pdf")
+		(tags "Resistor Axial_DIN0207 series Axial Horizontal pin pitch 10.16mm 0.25W = 1/4W length 6.3mm diameter 2.5mm")
+		(property "Reference" "R35"
+			(at 5.08 -2.37 0)
+			(layer "F.SilkS")
+			(effects
+				(font
+					(size 1 1)
+					(thickness 0.15)
+				)
+			)
+		)
+		(property "Value" "10k"
+			(at 5.08 2.37 0)
+			(layer "F.Fab")
+			(effects
+				(font
+					(size 1 1)
+					(thickness 0.15)
+				)
+			)
+		)
+		(property "Datasheet" ""
+			(at 0 0 0)
+			(layer "F.Fab")
+			(hide yes)
+			(effects
+				(font
+					(size 1.27 1.27)
+				)
+			)
+		)
+		(property "Description" ""
+			(at 0 0 0)
+			(layer "F.Fab")
+			(hide yes)
+			(effects
+				(font
+					(size 1.27 1.27)
+				)
+			)
+		)
+		(property "KiLib_Generator" "resistor/THT"
+			(at 0 0 0)
+			(layer "F.SilkS")
+			(hide yes)
+			(effects
+				(font
+					(size 1 1)
+					(thickness 0.15)
+				)
+			)
+		)
+		(attr through_hole)
+		(duplicate_pad_numbers_are_jumpers no)
+		(fp_line
+			(start 1.04 0)
+			(end 1.81 0)
+			(stroke
+				(width 0.12)
+				(type solid)
+			)
+			(layer "F.SilkS")
+		)
+		(fp_line
+			(start 9.12 0)
+			(end 8.35 0)
+			(stroke
+				(width 0.12)
+				(type solid)
+			)
+			(layer "F.SilkS")
+		)
+		(fp_rect
+			(start 1.81 -1.37)
+			(end 8.35 1.37)
+			(stroke
+				(width 0.12)
+				(type solid)
+			)
+			(fill no)
+			(layer "F.SilkS")
+		)
+		(fp_rect
+			(start -1.05 -1.5)
+			(end 11.21 1.5)
+			(stroke
+				(width 0.05)
+				(type solid)
+			)
+			(fill no)
+			(layer "F.CrtYd")
+		)
+		(fp_line
+			(start 0 0)
+			(end 1.93 0)
+			(stroke
+				(width 0.1)
+				(type solid)
+			)
+			(layer "F.Fab")
+		)
+		(fp_line
+			(start 10.16 0)
+			(end 8.23 0)
+			(stroke
+				(width 0.1)
+				(type solid)
+			)
+			(layer "F.Fab")
+		)
+		(fp_rect
+			(start 1.93 -1.25)
+			(end 8.23 1.25)
+			(stroke
+				(width 0.1)
+				(type solid)
+			)
+			(fill no)
+			(layer "F.Fab")
+		)
+		(fp_text user "${REFERENCE}"
+			(at 5.08 0 0)
+			(layer "F.Fab")
+			(effects
+				(font
+					(size 1 1)
+					(thickness 0.15)
+				)
+			)
+		)
+		(pad "1" thru_hole circle
+			(at 0 0)
+			(size 1.6 1.6)
+			(drill 0.8)
+			(layers "*.Cu" "*.Mask")
+			(remove_unused_layers no)
+			(net "+3V3")
+		)
+		(pad "2" thru_hole circle
+			(at 10.16 0)
+			(size 1.6 1.6)
+			(drill 0.8)
+			(layers "*.Cu" "*.Mask")
+			(remove_unused_layers no)
+			(net "SPARE_GPIO2")
+		)
+		(embedded_fonts no)
+		(model "${KICAD10_3DMODEL_DIR}/Resistor_THT.3dshapes/R_Axial_DIN0207_L6.3mm_D2.5mm_P10.16mm_Horizontal.step"
+			(offset
+				(xyz 0 0 0)
+			)
+			(scale
+				(xyz 1 1 1)
+			)
+			(rotate
+				(xyz 0 0 0)
+			)
 		)
 	)
@@
 		)
 	)
-	(footprint "Connector_JST:JST_XH_B6B-XH-A_1x06_P2.50mm_Vertical"
+	(footprint "Connector_JST:JST_XH_B7B-XH-A_1x07_P2.50mm_Vertical"
 		(layer "F.Cu")
 		(at 80.5 92)
-		(descr "JST XH series connector, B6B-XH-A (http://www.jst-mfg.com/product/pdf/eng/eXH.pdf)")
+		(descr "JST XH series connector, B7B-XH-A (http://www.jst-mfg.com/product/pdf/eng/eXH.pdf)")
 		(tags "connector JST XH vertical")
 		(property "Reference" "J8"
-			(at 6.25 -3.55 0)
+			(at 7.5 -3.55 0)
 			(layer "F.SilkS")
 			(effects
@@
 		)
 		(property "Value" "Winchman remote switches"
-			(at 6.25 4.6 0)
+			(at 7.5 4.6 0)
 			(layer "F.Fab")
 			(effects
@@
 		(fp_line
 			(start -1.8 2.75)
-			(end 6.25 2.75)
+			(end 7.5 2.75)
 			(stroke
 				(width 0.12)
@@
 		)
 		(fp_line
-			(start 14.3 -0.2)
-			(end 14.3 2.75)
-			(stroke
-				(width 0.12)
-				(type solid)
-			)
-			(layer "F.SilkS")
-		)
-		(fp_line
-			(start 14.3 2.75)
-			(end 6.25 2.75)
-			(stroke
-				(width 0.12)
-				(type solid)
-			)
-			(layer "F.SilkS")
-		)
-		(fp_line
-			(start 15.05 -0.2)
-			(end 14.3 -0.2)
+			(start 16.8 -0.2)
+			(end 16.8 2.75)
+			(stroke
+				(width 0.12)
+				(type solid)
+			)
+			(layer "F.SilkS")
+		)
+		(fp_line
+			(start 16.8 2.75)
+			(end 7.5 2.75)
+			(stroke
+				(width 0.12)
+				(type solid)
+			)
+			(layer "F.SilkS")
+		)
+		(fp_line
+			(start 17.55 -0.2)
+			(end 16.8 -0.2)
 			(stroke
 				(width 0.12)
@@
 		(fp_rect
 			(start -2.56 -2.46)
-			(end 15.06 3.51)
+			(end 17.56 3.51)
 			(stroke
 				(width 0.12)
@@
 		(fp_rect
 			(start 0.75 -2.45)
-			(end 11.75 -1.7)
-			(stroke
-				(width 0.12)
-				(type solid)
-			)
-			(fill no)
-			(layer "F.SilkS")
-		)
-		(fp_rect
-			(start 13.25 -2.45)
-			(end 15.05 -1.7)
+			(end 14.25 -1.7)
+			(stroke
+				(width 0.12)
+				(type solid)
+			)
+			(fill no)
+			(layer "F.SilkS")
+		)
+		(fp_rect
+			(start 15.75 -2.45)
+			(end 17.55 -1.7)
 			(stroke
 				(width 0.12)
@@
 		(fp_rect
 			(start -2.95 -2.85)
-			(end 15.45 3.9)
+			(end 17.95 3.9)
 			(stroke
 				(width 0.05)
@@
 		(fp_rect
 			(start -2.45 -2.35)
-			(end 14.95 3.4)
+			(end 17.45 3.4)
 			(stroke
 				(width 0.1)
@@
 		)
 		(fp_text user "${REFERENCE}"
-			(at 6.25 2.7 0)
+			(at 7.5 2.7 0)
 			(layer "F.Fab")
 			(effects
@@
 			(net "TENSION_RESET_SENSE")
 		)
+		(pad "7" thru_hole oval
+			(at 15 0)
+			(size 1.7 1.95)
+			(drill 0.95)
+			(layers "*.Cu" "*.Mask")
+			(remove_unused_layers no)
+			(net "SPARE_GPIO2")
+		)
 		(embedded_fonts no)
-		(model "${KICAD10_3DMODEL_DIR}/Connector_JST.3dshapes/JST_XH_B6B-XH-A_1x06_P2.50mm_Vertical.step"
+		(model "${KICAD10_3DMODEL_DIR}/Connector_JST.3dshapes/JST_XH_B7B-XH-A_1x07_P2.50mm_Vertical.step"
 			(offset
 				(xyz 0 0 0)

Commit message: kicad: bump board to rev 1.1, R35 routed
R35's pull-up traces (both pads) and J8 pin 7 routed by hand. DRC clean:
0 unconnected pads, only pre-existing unrelated warnings remain.
Routing:
- net SPARE_GPIO2: track 133.8 -> 214.5 mm, vias 6 -> 8
- net +3V3: track 406.9 -> 438.3 mm, vias 2 -> 4
Other:
- board text added: "Paraglider-tow-winch 1.1"
- board text removed: "Paraglider-tow-winch 1.0"
Changed lines of the file:
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@@
 	)
 	(paper "A2")
+	(title_block
+		(title "Tow Winch Mainboard - ESP32-S3 Control Node")
+		(date "2026-08-18")
+		(rev "1.1")
+		(comment 1 "PID tension control node: ESP32-S3, HX711 load cell amp header, Fardriver CAN, GIGA UART, USB-C program port")
+	)
 	(layers
 		(0 "F.Cu" signal)
@@
 		(layer "Edge.Cuts")
 	)
-	(gr_text "Paraglider-tow-winch 1.0"
+	(gr_text "Paraglider-tow-winch 1.1"
 		(at 45 109.5 0)
 		(layer "F.SilkS")
@@
 	)
 	(segment
+		(start 93 68)
+		(end 100 75)
+		(width 0.6)
+		(layer "F.Cu")
+		(net "+3V3")
+	)
+	(segment
 		(start 57.6 75.4)
 		(end 57.7 75.5)
@@
 	)
 	(segment
+		(start 90 68)
+		(end 93 68)
+		(width 0.6)
+		(layer "F.Cu")
+		(net "+3V3")
+	)
+	(segment
 		(start 32.5 62.75)
 		(end 32.5 68)
@@
 	)
 	(segment
+		(start 100 75)
+		(end 100 83)
+		(width 0.6)
+		(layer "F.Cu")
+		(net "+3V3")
+	)
+	(segment
 		(start 52.5 75.5)
 		(end 51.5 75.5)
@@
 	)
 	(segment
+		(start 79.5 68)
+		(end 84 68)
+		(width 0.6)
+		(layer "F.Cu")
+		(net "+3V3")
+	)
+	(segment
 		(start 59 70.5)
 		(end 57.6 71.9)
@@
 	)
 	(via
+		(at 84 68)
+		(size 0.8)
+		(drill 0.4)
+		(layers "F.Cu" "B.Cu")
+		(net "+3V3")
+	)
+	(via
+		(at 90 68)
+		(size 0.8)
+		(drill 0.4)
+		(layers "F.Cu" "B.Cu")
+		(net "+3V3")
+	)
+	(via
 		(at 52.5 75.5)
 		(size 0.8)
@@
 	)
 	(segment
+		(start 84 68)
+		(end 90 68)
+		(width 0.6)
+		(layer "B.Cu")
+		(net "+3V3")
+	)
+	(segment
 		(start 45 73)
 		(end 47.5 75.5)
@@
 	)
 	(segment
-		(start 93.565686 34.5)
+		(start 82.532843 45.532843)
 		(end 79.065686 49)
 		(width 0.2)
@@
 	)
 	(segment
+		(start 93.565686 34.5)
+		(end 82.532843 45.532843)
+		(width 0.2)
+		(layer "F.Cu")
+		(net "SPARE_GPIO2")
+	)
+	(segment
 		(start 70.5 49)
 		(end 70.5 54)
@@
 	)
 	(segment
+		(start 82.532843 45.532843)
+		(end 83.565686 44.5)
+		(width 0.2)
+		(layer "F.Cu")
+		(net "SPARE_GPIO2")
+	)
+	(segment
+		(start 100.66 73.5)
+		(end 110.16 83)
+		(width 0.2)
+		(layer "F.Cu")
+		(net "SPARE_GPIO2")
+	)
+	(segment
 		(start 33.5 59)
 		(end 54.5 59)
@@
 	)
 	(segment
+		(start 100.5 55.5)
+		(end 100.5 73.5)
+		(width 0.2)
+		(layer "F.Cu")
+		(net "SPARE_GPIO2")
+	)
+	(segment
 		(start 107.5 34.5)
 		(end 93.565686 34.5)
@@
 	)
 	(segment
+		(start 107 92)
+		(end 95.5 92)
+		(width 0.2)
+		(layer "F.Cu")
+		(net "SPARE_GPIO2")
+	)
+	(segment
 		(start 22.3125 65.5)
 		(end 24 65.5)
@@
 	)
 	(segment
+		(start 110.16 83)
+		(end 110.16 88.84)
+		(width 0.2)
+		(layer "F.Cu")
+		(net "SPARE_GPIO2")
+	)
+	(segment
+		(start 83.565686 44.5)
+		(end 97 44.5)
+		(width 0.2)
+		(layer "F.Cu")
+		(net "SPARE_GPIO2")
+	)
+	(segment
 		(start 54.5 59)
 		(end 56 57.5)
@@
 	)
 	(segment
+		(start 110.16 88.84)
+		(end 107 92)
+		(width 0.2)
+		(layer "F.Cu")
+		(net "SPARE_GPIO2")
+	)
+	(segment
+		(start 100.5 73.5)
+		(end 100.66 73.5)
+		(width 0.2)
+		(layer "F.Cu")
+		(net "SPARE_GPIO2")
+	)
+	(segment
 		(start 62 54.5)
 		(end 61.5 55)
@@
 	)
 	(via
+		(at 100.5 55.5)
+		(size 0.6)
+		(drill 0.3)
+		(layers "F.Cu" "B.Cu")
+		(net "SPARE_GPIO2")
+	)
+	(via
 		(at 61.5 57.5)
 		(size 0.6)
@@
 	)
 	(via
+		(at 97 44.5)
+		(size 0.6)
+		(drill 0.3)
+		(layers "F.Cu" "B.Cu")
+		(net "SPARE_GPIO2")
+	)
+	(via
 		(at 113 34.5)
 		(size 0.6)
@@
 	)
 	(segment
+		(start 97 52)
+		(end 100.5 55.5)
+		(width 0.2)
+		(layer "B.Cu")
+		(net "SPARE_GPIO2")
+	)
+	(segment
 		(start 30.5 59)
 		(end 33.5 59)
@@
 		(width 0.2)
 		(layer "B.Cu")
+		(net "SPARE_GPIO2")
+	)
+	(segment
+		(start 97 44.5)
+		(end 97 52)
+		(width 0.2)
+		(layer "B.Cu")
