File: kicad/winch_mainboard/winch_mainboard.kicad_sch (KiCad schematic)
At the start: 35 parts, among them J1 PWR_IN_24V (from Victron 96V-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, J10 Heltec WiFi LoRa 32 V4 - Head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, J11 Heltec WiFi LoRa 32 V4 - Head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, J12 Hall sensors (drum direction), J2 CAN_BUS (to Fardriver), J3 To GIGA UART (TXD,RXD,GND), J4 HX711 module (3V3,GND,DT,SCK), J6 Spare I/O, J7 Line cut switch (winch), J8 Winchman remote switches, J9 Cut motor out (24V) - A/B = K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, K1 Relay 24V coil (Songle SRD-24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, Q1 BC337-40, U1 ESP32-S3 N16R8 DevKitC-1, U3 SN65HVD230

Commit message: update
Parts:
- J4: value HX711 module (3V3,GND,DT,SCK) -> HX711 module, flat-mount socket (GND,DT,SCK,3V3); footprint Connector_JST:JST_XH_B4B-XH-A_1x04_P2.50mm_Vertical -> Connector_PinSocket_2.54mm:PinSocket_1x04_P2.54mm_Vertical
- J9: value Cut motor out (24V) - A/B = K1 contacts, verify NO before wiring -> Cut motor out (24V) - 1/2=K1 contacts A/B (verify NO), 3=GND
Connections:
- net +3V3: now also J4.4 (Pin_4); no longer J4.1 (Pin_1)
- net GND: now also J4.1 (Pin_1); no longer J4.2 (Pin_2)
- net HX711_DT: now also J4.2 (Pin_2); no longer J4.3 (Pin_3)
- net HX711_SCK: now also J4.3 (Pin_3); no longer J4.4 (Pin_4)
Changed lines of the file:
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@@
 	)
 	(label "HX711_DT"
-		(at 312.42 201.93 0)
+		(at 312.42 199.39 0)
 		(effects
 			(font
@@
 	)
 	(label "HX711_SCK"
-		(at 312.42 204.47 0)
+		(at 312.42 201.93 0)
 		(effects
 			(font
@@
 	(symbol
 		(lib_id "power:+3V3")
-		(at 312.42 196.85 0)
+		(at 312.42 204.47 0)
 		(unit 1)
 		(exclude_from_sim no)
@@
 		(dnp no)
 		(property "Reference" "#PWR026"
-			(at 312.42 199.85 0)
+			(at 312.42 207.47 0)
 			(hide yes)
 			(effects
@@
 		)
 		(property "Value" "+3V3"
-			(at 312.62 194.35 0)
+			(at 312.62 201.97 0)
 			(effects
 				(font
@@
 		)
 		(property "Footprint" ""
-			(at 312.42 196.85 0)
+			(at 312.42 204.47 0)
 			(hide yes)
 			(effects
@@
 		)
 		(property "Datasheet" ""
-			(at 312.42 196.85 0)
+			(at 312.42 204.47 0)
 			(hide yes)
 			(effects
@@
 	(symbol
 		(lib_id "power:GND")
-		(at 312.42 199.39 0)
+		(at 312.42 196.85 0)
 		(unit 1)
 		(exclude_from_sim no)
@@
 		(dnp no)
 		(property "Reference" "#PWR027"
-			(at 312.42 202.39 0)
+			(at 312.42 199.85 0)
 			(hide yes)
 			(effects
@@
 		)
 		(property "Value" "GND"
-			(at 312.62 196.89 0)
+			(at 312.62 194.35 0)
 			(effects
 				(font
@@
 		)
 		(property "Footprint" ""
-			(at 312.42 199.39 0)
+			(at 312.42 196.85 0)
 			(hide yes)
 			(effects
@@
 		)
 		(property "Datasheet" ""
-			(at 312.42 199.39 0)
+			(at 312.42 196.85 0)
 			(hide yes)
 			(effects
@@
 			)
 		)
-		(property "Value" "HX711 module (3V3,GND,DT,SCK)"
+		(property "Value" "HX711 module, flat-mount socket (GND,DT,SCK,3V3)"
 			(at 320.04 202.39 0)
 			(effects
@@
 			)
 		)
-		(property "Footprint" "Connector_JST:JST_XH_B4B-XH-A_1x04_P2.50mm_Vertical"
+		(property "Footprint" "Connector_PinSocket_2.54mm:PinSocket_1x04_P2.54mm_Vertical"
 			(at 320.04 199.39 0)
 			(hide yes)
@@
 			)
 		)
-		(property "Value" "Cut motor out (24V) - A/B = K1 contacts, verify NO before wiring"
+		(property "Value" "Cut motor out (24V) - 1/2=K1 contacts A/B (verify NO), 3=GND"
 			(at 190.5 348.44 0)
 			(effects

Commit message: kicad: widen winchman remote (J8) to 7 pins for a proper release-switch pull-up, replacing the planned hand-wired bodge
J8 was full at 6/6 pins, so the release switch (added last session as a
firmware-only GPIO2 target) had no clean way to get a real pull-up like
the other four winchman-remote switches. Instead of the planned hand-wired
jumper off J6's spare pin, widened J8 to a 7-pin JST-XH connector and
added R35 (10k, +3V3 to SPARE_GPIO2/GPIO2) - same convention as R31-R34.

New Conn_01x07 schematic symbol (extended from the stock Conn_01x06
pattern, same pin pitch). PCB footprint swapped to the stock
JST_XH_B7B-XH-A_1x07; pins 1-6 keep identical physical positions so
existing routed copper is untouched. R35 placed at a location verified
clear of existing traces/footprints (an earlier attempt at a more
"obvious" spot turned out to short against an existing TENSION_RESET_SENSE
trace - moved after DRC caught it). back_gnd zone refilled to account for
the 3 new pads. ERC/DRC clean except pre-existing warnings and the 3 new
unrouted connections, left for manual routing as usual.

Also: .gitignore now excludes *.lck (KiCad's own transient lock files,
were being churned in/out of git status on every open/close).
Parts:
- added R35: 10k, Resistor_THT:R_Axial_DIN0207_L6.3mm_D2.5mm_P10.16mm_Horizontal, symbol Device:R
- J8: footprint Connector_JST:JST_XH_B6B-XH-A_1x06_P2.50mm_Vertical -> Connector_JST:JST_XH_B7B-XH-A_1x07_P2.50mm_Vertical; symbol Connector_Generic:Conn_01x06 -> Connector_Generic:Conn_01x07
Connections:
- net +3V3: now also R35.1
- net SPARE_GPIO2: now also J8.7 (Pin_7), R35.2
Changed lines of the file:
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@@
 	(wire
 		(pts
+			(xy 25.4 365.76) (xy 22.86 365.76)
+		)
+		(stroke
+			(width 0)
+			(type default)
+		)
+	)
+	(label "SPARE_GPIO2"
+		(at 22.86 365.76 0)
+		(effects
+			(font
+				(size 1.27 1.27)
+			)
+			(justify left bottom)
+		)
+	)
+	(wire
+		(pts
 			(xy 54.61 351.79) (xy 54.61 349.25)
 		)
@@
 		)
 	)
+	(symbol
+		(lib_id "Device:R")
+		(at 530.86 350.52 0)
+		(unit 1)
+		(exclude_from_sim no)
+		(in_bom yes)
+		(on_board yes)
+		(dnp no)
+		(property "Reference" "R35"
+			(at 530.86 347.52 0)
+			(effects
+				(font
+					(size 1.27 1.27)
+				)
+			)
+		)
+		(property "Value" "10k"
+			(at 530.86 353.52 0)
+			(effects
+				(font
+					(size 1.27 1.27)
+				)
+			)
+		)
+		(property "Footprint" "Resistor_THT:R_Axial_DIN0207_L6.3mm_D2.5mm_P10.16mm_Horizontal"
+			(at 530.86 350.52 0)
+			(hide yes)
+			(effects
+				(font
+					(size 1.27 1.27)
+				)
+			)
+		)
+		(property "Datasheet" ""
+			(at 530.86 350.52 0)
+			(hide yes)
+			(effects
+				(font
+					(size 1.27 1.27)
+				)
+			)
+		)
+		(pin "1"
+		)
+		(pin "2"
+		)
+		(instances
+			(project "winch_mainboard"
+				(path "/8f1a2b3c-4d5e-4a6b-9c7d-1e2f3a4b5c6d"
+					(reference "R35")
+					(unit 1)
+				)
+			)
+		)
+	)
+	(symbol
+		(lib_id "power:+3V3")
+		(at 530.86 344.17 0)
+		(unit 1)
+		(exclude_from_sim no)
+		(in_bom yes)
+		(on_board yes)
+		(dnp no)
+		(property "Reference" "#PWR050"
+			(at 530.86 347.17 0)
+			(hide yes)
+			(effects
+				(font
+					(size 1.27 1.27)
+				)
+			)
+		)
+		(property "Value" "+3V3"
+			(at 531.06 341.67 0)
+			(effects
+				(font
+					(size 1.27 1.27)
+				)
+			)
+		)
+		(property "Footprint" ""
+			(at 530.86 344.17 0)
+			(hide yes)
+			(effects
+				(font
+					(size 1.27 1.27)
+				)
+			)
+		)
+		(property "Datasheet" ""
+			(at 530.86 344.17 0)
+			(hide yes)
+			(effects
+				(font
+					(size 1.27 1.27)
+				)
+			)
+		)
+		(pin "1"
+		)
+		(instances
+			(project "winch_mainboard"
+				(path "/8f1a2b3c-4d5e-4a6b-9c7d-1e2f3a4b5c6d"
+					(reference "#PWR050")
+					(unit 1)
+				)
+			)
+		)
+	)
+	(wire
+		(pts
+			(xy 530.86 346.71) (xy 530.86 344.17)
+		)
+		(stroke
+			(width 0)
+			(type default)
+		)
+	)
+	(wire
+		(pts
+			(xy 530.86 354.33) (xy 530.86 356.87)
+		)
+		(stroke
+			(width 0)
+			(type default)
+		)
+	)
+	(label "SPARE_GPIO2"
+		(at 530.86 356.87 0)
+		(effects
+			(font
+				(size 1.27 1.27)
+			)
+			(justify left bottom)
+		)
+	)
 	(wire
 		(pts
@@
 	)
 	(symbol
-		(lib_id "Connector_Generic:Conn_01x06")
+		(lib_id "Connector_Generic:Conn_01x07")
 		(at 30.48 355.6 0)
 		(unit 1)
@@
 			)
 		)
-		(property "Footprint" "Connector_JST:JST_XH_B6B-XH-A_1x06_P2.50mm_Vertical"
+		(property "Footprint" "Connector_JST:JST_XH_B7B-XH-A_1x07_P2.50mm_Vertical"
 			(at 30.48 355.6 0)
 			(hide yes)
@@
 		(pin "6"
 		)
+		(pin "7"
+		)
 		(instances
